Commit message: Update puzzlebot.xacro

File: Challenges_P2/simulation_puzzlebot_ws/puzzlebot_queza/urdf/puzzlebot.xacro (robot description, xacro)
@@ -3,5 +3,5 @@
   <xacro:property name="package_name" value="puzzlebot_queza"/>
   <xacro:property name="PI" value="3.14159265"/>
-  <xacro:property name="wheelSeparation" value="0.20"/>
+  <xacro:property name="wheelSeparation" value="0.189"/>
   <xacro:property name="wheelDiameter" value="0.10"/>
   <xacro:property name="wheelThickness" value="0.008"/>
@@ -76,7 +76,7 @@
     </collision>
     <inertial>
-      <origin xyz="0 0 ${wheelDiameter-base_elevation}" rpy="0 0 0"/>
-      <mass value="10"/>
-      <inertia ixx="0.333333" ixy="0.0" ixz="0.0"  iyy="0.333333" iyz="0.0"  izz="0.6" />
+      <origin xyz="-0.0550 0 0" rpy="0 0 0"/>
+      <mass value="1.485"/>
+      <inertia ixx="0.00576" ixy="0.0" ixz="0.0" iyy="0.00347" iyz="0.0" izz="0.00862" />
     </inertial>
   </link>
@@ -292,6 +292,6 @@
     <inertial>
       <origin xyz="0 0 0" />
-      <mass value="5" />
-      <inertia ixx="0.0135417" ixy="0.0" ixz="0.0"  iyy="0.0135417" iyz="0.0"  izz="0.025" />
+      <mass value="0.056" />
+      <inertia ixx="0.000035" ixy="0.0" ixz="0.0" iyy="0.00007" iyz="0.0" izz="0.000035" />
     </inertial>
   </link>
@@ -318,6 +318,6 @@
     <inertial>
       <origin xyz="0 0 0" />
-      <mass value="5" />
-      <inertia ixx="0.0135417" ixy="0.0" ixz="0.0"  iyy="0.0135417" iyz="0.0"  izz="0.025" />
+      <mass value="0.056" />
+      <inertia ixx="0.000035" ixy="0.0" ixz="0.0" iyy="0.00007" iyz="0.0" izz="0.000035" />
     </inertial>
   </link>
@@ -342,6 +342,10 @@
     </collision>
     <inertial>
-      <mass value="0.1"/>
-      <inertia ixx="0.000009" ixy="0" ixz="0" iyy="0.000009" iyz="0" izz="0.000009"/>
+      <mass value="0.01"/>
+      <origin xyz="0 0 0" rpy="0 0 0"/>
+      <inertia
+        ixx="0.000000625" ixy="0" ixz="0"
+        iyy="0.000000625" iyz="0"
+        izz="0.000000625"/>
     </inertial>
   </link>
@@ -431,6 +435,6 @@
       <max_linear_acceleration>0.5</max_linear_acceleration>
       <min_linear_acceleration>-0.5</min_linear_acceleration>
-      <max_angular_acceleration>1</max_angular_acceleration>
-      <min_angular_acceleration>-1</min_angular_acceleration>
+      <max_angular_acceleration>2</max_angular_acceleration>
+      <min_angular_acceleration>-2</min_angular_acceleration>
       <max_linear_velocity>0.5</max_linear_velocity>
       <min_linear_velocity>-0.3</min_linear_velocity>
@@ -443,3 +447,9 @@
     </plugin>
   </gazebo>
+  <gazebo reference="$(arg ns)/caster_wheel_link">
+    <mu1>0.01</mu1>
+    <mu2>0.01</mu2>
+    <kp>1000000.0</kp>
+    <kd>1.0</kd>
+  </gazebo>
 </robot>
